File: PCB/neuztech-4.sch (EAGLE design)
At the start: 77 parts, among them IC1 DSPIC30F3013-30I/SP, IC2 TL074P, IC4 ICL7660CPA, IC5 MCP4822-E/P, IC6 MCP4822-E/P, IC7 7805TV, SW1 SK-22D01

Commit message: Add 16 pin header, remove battery power distribution
Parts:
- removed C15: 10uF, rcl:CPOL-USE2-4
- removed D11, D12, D7, D8: 1N4148DO35-7, diode:1N4148DO35-7
- removed G1: AB9V, battery:AB9V
- removed IC4: ICL7660CPA, maxim:ICL7660CPA
- removed IC7: 7805TV, linear:7805TV
- removed SV2: EURO_POWER_HEADERFAT_PADS, MusicThingModular:EURO_POWER_HEADERFAT_PADS
- removed SW1: SK-22D01, ptrz:SK-22D01
- added D1, D2, D3: 1N5819-B, diode:1N5819-B
- added U$1: POWER, eurorack:POWER
Connections:
- removed net N$36: C15.+, IC4.CAP+
- removed net N$38: C15.-, IC4.CAP-
- removed net N$39: IC4.VOUT, SW1.NC2
- removed net N$40: G1.+, SW1.C
- removed net N$41: D11.A, SW1.NC
- removed net N$42: D12.C, SW1.C2
- new net N$9: D3.A, U$1.+5V
- net +12V: now also D1.C; no longer D11.C, D7.C, IC4.V+, IC7.VI
- net +5V: now also D3.C; no longer IC7.VO
- net -12V: now also D2.A; no longer D12.A, D8.A
- net GND: now also U$1.GND; no longer G1.-, IC4.GND, IC7.GND, SV2.3, SV2.4, SV2.5, SV2.6, SV2.7, SV2.8
- net N$15: now also D2.C, U$1.-12V; no longer D8.C, SV2.1, SV2.2
- net N$25: now also D1.A, U$1.+12V; no longer D7.A, SV2.10, SV2.9
