File: PCB/neuztech-4.brd (EAGLE design)
At the start: 69.8 x 106.5 mm, 77 parts, among them IC1 DSPIC30F3013-30I/SP, IC2 TL074P, IC4 ICL7660CPA, IC5 MCP4822-E/P, IC6 MCP4822-E/P, IC7 7805TV, SW1 SK-22D01

Commit message: Add 16 pin header, remove battery power distribution
Parts:
- removed C15: 10uF, rcl:E2-4
- removed D11, D12, D7, D8: 1N4148DO35-7, diode:DO35-7
- removed G1: AB9V, battery:AB9V
- removed IC4: ICL7660CPA, maxim:DIL08
- removed IC7: 7805TV, linear:TO220V
- removed SV2: EURO_POWER_HEADERFAT_PADS, MusicThingModular:EURO_PWR_HEADER_FAT
- removed SW1: SK-22D01, ptrz:SK-22D01-MG
- added D1, D2, D3: 1N5819-B, diode:DO41-7.6
- added U$1: POWER, eurorack:POWER_16
Connections:
- removed net N$36: C15.+, IC4.2
- removed net N$38: C15.-, IC4.4
- removed net N$39: IC4.5, SW1.NC2
- removed net N$40: G1.+, SW1.C1
- removed net N$41: D11.A, SW1.NC1
- removed net N$42: D12.C, SW1.C2
- new net N$9: D3.A, U$1.11, U$1.12
- net +12V: now also D1.C; no longer D11.C, D7.C, IC4.8, IC7.1
- net +5V: now also D3.C; no longer IC7.3
- net -12V: now also D2.A; no longer D12.A, D8.A
- net GND: now also U$1.3, U$1.4, U$1.5, U$1.6, U$1.7, U$1.8; no longer G1.-, IC4.3, IC7.2, SV2.3, SV2.4, SV2.5, SV2.6, SV2.7, SV2.8
- net N$15: now also D2.C, U$1.1, U$1.2; no longer D8.C, SV2.1, SV2.2
- net N$25: now also D1.A, U$1.10, U$1.9; no longer D7.A, SV2.10, SV2.9
Routing:
- net +12V: track 154.0 -> 81.4 mm, vias 11 -> 8
- net N$41: track 39.9 -> 0.00 mm, vias 2 -> 0
- net N$42: track 39.6 -> 0.00 mm, vias 1 -> 0
- net N$9: track 0.00 -> 39.3 mm
- net N$39: track 35.9 -> 0.00 mm, vias 1 -> 0
- net N$40: track 21.4 -> 0.00 mm, vias 2 -> 0
- net N$36: track 13.0 -> 0.00 mm
- net N$38: track 9.39 -> 0.00 mm
- net N$44: track 70.3 -> 63.2 mm
- net N$2: track 6.50 -> 0.00 mm
- net N$24: track 113.6 -> 109.4 mm
- net +5V: track 291.1 -> 294.0 mm
- net GND: track 0.00 -> 2.64 mm, vias 17 -> 15
- net N$15: track 6.91 -> 8.77 mm
- net N$25: track 6.12 -> 7.81 mm
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Other:
- outline, holes or cut-outs redrawn
- board text removed: "7660"
- board text removed: "OFF"

Commit message: Rearrange components, Generate new gerbers, Update readme
Parts:
- moved D1 15.3 mm to (24.0, 86.5), turned to 180 degrees
- moved U$1 0.71 mm to (12.5, 99.5)
Routing:
- net +12V: track 81.4 -> 68.0 mm, vias 8 -> 6
- net N$25: track 7.81 -> 18.8 mm, vias 0 -> 2
Other:
- board text removed: "ON"
Changed lines of the file:
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@@
 <layer number="24" name="bOrigins" color="15" fill="1" visible="yes" active="yes"/>
 <layer number="25" name="tNames" color="7" fill="1" visible="no" active="yes"/>
-<layer number="26" name="bNames" color="7" fill="1" visible="no" active="yes"/>
+<layer number="26" name="bNames" color="7" fill="1" visible="yes" active="yes"/>
 <layer number="27" name="tValues" color="7" fill="1" visible="no" active="yes"/>
 <layer number="28" name="bValues" color="7" fill="1" visible="no" active="yes"/>
@@
 <text x="4.1" y="97.1" size="0.8128" layer="26" rot="MR270">RED STRIPE</text>
 <text x="56.9" y="19.8" size="1.778" layer="30" ratio="17" rot="MR0">V1.2</text>
-<text x="19.7" y="101.5" size="1.5" layer="26" font="vector" rot="SMR0">ON</text>
 <text x="44.7" y="20.9" size="1.4" layer="25" font="vector">TALL
 TRIMMER</text>
@@
 <attribute name="VALUE" x="38.76291875" y="45.05445" size="2.09043125" layer="27" ratio="10" rot="SR0"/>
 </element>
-<element name="U$1" library="eurorack" package="POWER_16" value="POWER" x="12" y="100" smashed="yes" rot="MR180">
-<attribute name="NAME" x="24.88" y="102.825" size="1.27" layer="26" ratio="10" rot="MR180"/>
-</element>
-<element name="D1" library="diode" library_urn="urn:adsk.eagle:library:210" package="DO41-7.6" package3d_urn="urn:adsk.eagle:package:43421/1" value="1N5819-B" x="12" y="96" smashed="yes">
-<attribute name="NAME" x="9.968" y="97.651" size="1.27" layer="25" ratio="10"/>
-<attribute name="POPULARITY" value="11" x="12" y="96" size="1.778" layer="27" display="off"/>
-<attribute name="VALUE" x="9.968" y="93.079" size="1.27" layer="27" ratio="10"/>
+<element name="U$1" library="eurorack" package="POWER_16" value="POWER" x="12.5" y="99.5" smashed="yes" rot="MR180"/>
+<element name="D1" library="diode" library_urn="urn:adsk.eagle:library:210" package="DO41-7.6" package3d_urn="urn:adsk.eagle:package:43421/1" value="1N5819-B" x="24" y="86.5" smashed="yes" rot="R180">
+<attribute name="NAME" x="26.032" y="84.849" size="1.27" layer="25" ratio="10" rot="R180"/>
+<attribute name="POPULARITY" value="11" x="24" y="86.5" size="1.778" layer="27" rot="R180" display="off"/>
+<attribute name="VALUE" x="26.032" y="89.421" size="1.27" layer="27" ratio="10" rot="R180"/>
 </element>
 <element name="D2" library="diode" library_urn="urn:adsk.eagle:library:210" package="DO41-7.6" package3d_urn="urn:adsk.eagle:package:43421/1" value="1N5819-B" x="5" y="91.5" smashed="yes" rot="R270">
@@
 <wire x1="17.4752" y1="39.0144" x2="17.325" y2="38.98" width="0.4064" layer="1"/>
 <wire x1="21.5392" y1="39.0144" x2="22.129" y2="38.935" width="0.4064" layer="16"/>
-<wire x1="11.7856" y1="89.408" x2="8.128" y2="93.0656" width="0.4064" layer="16"/>
-<wire x1="17.0688" y1="84.1248" x2="11.7856" y2="89.408" width="0.4064" layer="1"/>
-<wire x1="16.6624" y1="83.7184" x2="17.0688" y2="84.1248" width="0.4064" layer="1"/>
-<wire x1="17.4752" y1="82.9056" x2="16.6624" y2="83.7184" width="0.4064" layer="16"/>
-<wire x1="19.9136" y1="82.9056" x2="17.4752" y2="82.9056" width="0.4064" layer="16"/>
-<wire x1="23.1648" y1="79.6544" x2="21.5392" y2="81.28" width="0.4064" layer="16"/>
-<wire x1="21.5392" y1="81.28" x2="19.9136" y2="82.9056" width="0.4064" layer="16"/>
-<wire x1="23.1648" y1="76.8096" x2="23.1648" y2="79.6544" width="0.4064" layer="16"/>
+<wire x1="23.1648" y1="79.94914375" x2="23.1648" y2="76.8096" width="0.4064" layer="16"/>
 <wire x1="21.9456" y1="75.5904" x2="23.1648" y2="76.8096" width="0.4064" layer="16"/>
 <wire x1="21.9456" y1="72.3392" x2="21.9456" y2="75.5904" width="0.4064" layer="16"/>
@@
 <wire x1="25.1968" y1="69.9008" x2="25.146153125" y2="69.765340625" width="0.4064" layer="16"/>
 <via x="19.1008" y="40.64" extent="1-16" drill="0.4064"/>
-<via x="11.7856" y="89.408" extent="1-16" drill="0.4064"/>
-<via x="16.6624" y="83.7184" extent="1-16" drill="0.4064"/>
 <via x="21.9456" y="72.3392" extent="1-16" drill="0.4064"/>
 <via x="19.9136" y="44.2976" extent="1-16" drill="0.4064"/>
@@
 <via x="31.2928" y="67.056" extent="1-16" drill="0.4064"/>
 <contactref element="D1" pad="C"/>
-<wire x1="8.128" y1="95.938" x2="8.19" y2="96" width="0.4064" layer="16"/>
-<wire x1="8.128" y1="93.0656" x2="8.128" y2="95.938" width="0.4064" layer="16"/>
+<wire x1="26.36" y1="83.05" x2="23.60394375" y2="83.05" width="0.4064" layer="16"/>
+<wire x1="23.60394375" y1="83.05" x2="22.36" y2="81.80605625" width="0.4064" layer="16"/>
+<wire x1="22.36" y1="81.80605625" x2="22.36" y2="80.75394375" width="0.4064" layer="16"/>
+<wire x1="22.36" y1="80.75394375" x2="23.1648" y2="79.94914375" width="0.4064" layer="16"/>
+<wire x1="27.81" y1="86.5" x2="27.81" y2="84.5" width="0.4064" layer="16"/>
+<wire x1="27.81" y1="84.5" x2="26.36" y2="83.05" width="0.4064" layer="16"/>
 </signal>
 <signal name="N$61">
@@
 <contactref element="U$1" pad="2"/>
 <contactref element="D2" pad="C"/>
-<wire x1="5.65" y1="101.27" x2="5.65" y2="95.96" width="0.4064" layer="16"/>
-<wire x1="5.65" y1="95.96" x2="5" y2="95.31" width="0.4064" layer="16"/>
-<wire x1="5.65" y1="98.73" x2="5.65" y2="101.27" width="0.4064" layer="1"/>
+<wire x1="6.15" y1="100.77" x2="6.15" y2="96.46" width="0.4064" layer="16"/>
+<wire x1="6.15" y1="96.46" x2="5" y2="95.31" width="0.4064" layer="16"/>
+<wire x1="6.15" y1="98.23" x2="6.15" y2="100.77" width="0.4064" layer="1"/>
 </signal>
 <signal name="N$25">
@@
 <contactref element="U$1" pad="9"/>
 <contactref element="D1" pad="A"/>
-<wire x1="15.81" y1="96" x2="15.81" y2="101.27" width="0.4064" layer="16"/>
-<wire x1="15.81" y1="98.73" x2="15.81" y2="101.27" width="0.4064" layer="1"/>
+<wire x1="16.31" y1="100.77" x2="16.31" y2="95.77" width="0.4064" layer="16"/>
+<wire x1="16.31" y1="95.77" x2="15.81" y2="95.27" width="0.4064" layer="16"/>
+<wire x1="20.19" y1="90.89" x2="20.19" y2="86.5" width="0.4064" layer="16"/>
+<wire x1="16.31" y1="98.23" x2="16.31" y2="100.77" width="0.4064" layer="1"/>
+<via x="15.81" y="95.27" extent="1-16" drill="0.4064"/>
+<wire x1="15.81" y1="95.27" x2="20.19" y2="90.89" width="0.4064" layer="1"/>
+<via x="20.19" y="90.89" extent="1-16" drill="0.4064"/>
 </signal>
 <signal name="N$34">
@@
 <wire x1="32.9184" y1="97.0816" x2="31.5" y2="98.5" width="0.4064" layer="16"/>
 <wire x1="29" y1="98.5" x2="31.5" y2="98.5" width="0.4064" layer="16"/>
-<wire x1="20.7224" y1="95.5" x2="26" y2="95.5" width="0.4064" layer="16"/>
-<wire x1="11.7856" y1="86.5632" x2="20.7224" y2="95.5" width="0.4064" layer="16"/>
-<wire x1="26" y1="95.5" x2="29" y2="98.5" width="0.4064" layer="16"/>
+<wire x1="20.2224" y1="95" x2="25.5" y2="95" width="0.4064" layer="16"/>
+<wire x1="11.7856" y1="86.5632" x2="20.2224" y2="95" width="0.4064" layer="16"/>
+<wire x1="25.5" y1="95" x2="29" y2="98.5" width="0.4064" layer="16"/>
 </signal>
 <signal name="N$45">
@@
 <contactref element="U$1" pad="11"/>
 <contactref element="D3" pad="A"/>
-<wire x1="18.35" y1="98.73" x2="18.35" y2="97.65" width="0.4064" layer="16"/>
-<wire x1="19.5" y1="96.5" x2="25" y2="96.5" width="0.4064" layer="16"/>
-<wire x1="25" y1="96.5" x2="28.5" y2="100" width="0.4064" layer="16"/>
+<wire x1="18.85" y1="98.23" x2="18.85" y2="97.15" width="0.4064" layer="16"/>
+<wire x1="20" y1="96" x2="24.5" y2="96" width="0.4064" layer="16"/>
+<wire x1="24.5" y1="96" x2="28.5" y2="100" width="0.4064" layer="16"/>
 <wire x1="28.5" y1="100" x2="49" y2="100" width="0.4064" layer="16"/>
 <wire x1="49" y1="100" x2="50" y2="99" width="0.4064" layer="16"/>
 <wire x1="50" y1="99" x2="51.69" y2="99" width="0.4064" layer="16"/>
-<wire x1="18.35" y1="97.65" x2="19.5" y2="96.5" width="0.4064" layer="16"/>
-<wire x1="18.35" y1="98.73" x2="18.35" y2="101.27" width="0.4064" layer="1"/>
+<wire x1="18.85" y1="97.15" x2="20" y2="96" width="0.4064" layer="16"/>
+<wire x1="18.85" y1="98.23" x2="18.85" y2="100.77" width="0.4064" layer="1"/>
 </signal>
 </signals>
